Commit message: refactor and node combine

File: ws/src/Universal_Robots_ROS2_Driver/ur_robot_driver/urdf/ur.ros2_control.xacro (robot description, xacro)
@@ -299,5 +299,5 @@
       <hardware>
         <plugin>feetech_ros2_driver/FeetechHardwareInterface</plugin>
-        <param name="usb_port">/dev/ttyUSB0</param>
+        <param name="usb_port">/dev/feetech_driver</param>
       </hardware>
       <joint name="left_finger_joint">

File: ws/src/Universal_Robots_ROS2_Driver/ur_robot_driver/urdf/ur.urdf.xacro (robot description, xacro)
@@ -101,5 +101,6 @@
   <xacro:include filename="$(find realsense2_description)/urdf/_d435.urdf.xacro" />
   <xacro:sensor_d435 parent="tool0" use_nominal_extrinsics="$(arg use_nominal_extrinsics)" add_plug="$(arg add_plug)" use_mesh="$(arg use_mesh)">
-    <origin xyz="0.03 0 0.015" rpy="0 -1.57 3.14"/>
+    <!-- <origin xyz="0.03 0 0.015" rpy="0 -1.57 3.14"/> -->
+    <origin xyz="0.03 0 0.01" rpy="0 -1.57 3.14"/>
   </xacro:sensor_d435>
 </robot>
