Commit message: new gripper prismatic urdf behaviour

File: ws/src/Universal_Robots_ROS2_Driver/ur_moveit_config/srdf/ur_macro.srdf.xacro (robot description, xacro)
@@ -15,5 +15,5 @@
     </group>
     <group name="gripper_group">
-      <joint name="left_finger_joint"/>
+      <joint name="joint_finger_left"/>
     </group>
     <!--GROUP STATES - Purpose - Define a named state for a particular group, in terms of joint values. This is useful to define states like 'folded arms'-->
@@ -43,5 +43,5 @@
     </group_state>
     <!--END EFFECTOR - Purpose - Represent information about an end effector.-->
-    <end_effector name="scissors_gripper" parent_link="tool0" group="gripper_group" parent_group="ur_manipulator"/>
+    <end_effector name="parallel_gripper" parent_link="tool0" group="gripper_group" parent_group="ur_manipulator"/>
     <!--VIRTUAL JOINT - Purpose - this element defines a virtual joint between a robot link and an external frame of reference (considered fixed with respect to the robot)-->
     <!--DISABLE COLLISIONS - By default it is assumed that any link of the robot could potentially come into collision with any other link in the robot. This tag disables collision checking between a specified pair of links. -->
@@ -57,7 +57,7 @@
     <disable_collisions link1="wrist_1_link" link2="wrist_3_link" reason="Never" />
     <disable_collisions link1="wrist_2_link" link2="wrist_3_link" reason="Adjacent" />
-    <disable_collisions link1="gripper_base_link" link2="left_finger_link" reason="Adjacent"/>
-    <disable_collisions link1="gripper_base_link" link2="right_finger_link" reason="Adjacent"/>
-    <disable_collisions link1="left_finger_link" link2="right_finger_link" reason="Never"/>
+    <disable_collisions link1="gripper_base_link" link2="link_finger_left" reason="Adjacent"/>
+    <disable_collisions link1="gripper_base_link" link2="link_finger_right" reason="Adjacent"/>
+    <disable_collisions link1="link_finger_left" link2="link_finger_right" reason="Never"/>
     <disable_collisions link1="gripper_base_link" link2="flange" reason="Never"/>
     <disable_collisions link1="gripper_base_link" link2="tool0" reason="Never"/>

File: ws/src/Universal_Robots_ROS2_Driver/ur_robot_driver/urdf/scissors_gripper.urdf.xacro (robot description, xacro)
@@ -33,5 +33,5 @@
     <origin xyz="0 -0.04 0.06" rpy="0 0 0"/>
     <axis xyz="1 0 0"/>
-    <limit lower="0.0" upper="0.5" effort="5.0" velocity="3.0"/>
+    <limit lower="0.942478" upper="2.21657" effort="5.0" velocity="3.0"/>
   </joint>
   <link name="left_finger_link">
@@ -60,5 +60,5 @@
     <axis xyz="1 0 0"/>
     <mimic joint="left_finger_joint" multiplier="-1.0"/>
-    <limit lower="-0.5" upper="0.0" effort="5.0" velocity="3.0"/>
+    <limit lower="-2.21657" upper="0.942478" effort="5.0" velocity="3.0"/>
   </joint>
   <link name="right_finger_link">

File: ws/src/Universal_Robots_ROS2_Driver/ur_robot_driver/urdf/ur.ros2_control.xacro (robot description, xacro)
@@ -296,13 +296,13 @@
       </gpio>
     </ros2_control>
-    <ros2_control name="ScissorsGripperControl" type="system">
+    <ros2_control name="ParallelGripperControl" type="system">
       <hardware>
         <plugin>feetech_ros2_driver/FeetechHardwareInterface</plugin>
-        <param name="usb_port">/dev/feetech_driver</param>
+        <param name="usb_port">/dev/ttyACM0</param>
       </hardware>
-      <joint name="left_finger_joint">
+      <joint name="joint_finger_left">
         <param name="id">1</param>
-        <param name="range_min">0.0</param>
-        <param name="range_max">0.5</param>
+        <param name="range_min">2620</param>
+        <param name="range_max">3791</param>
         <command_interface name="position"/>
         <state_interface name="position"/>

File: ws/src/Universal_Robots_ROS2_Driver/ur_robot_driver/urdf/ur.urdf.xacro (robot description, xacro)
@@ -4,5 +4,5 @@
   <xacro:arg name="name" default="ur"/>
   <xacro:include filename="$(find ur_description)/urdf/ur_macro.xacro"/>
-  <xacro:include filename="$(find ur_robot_driver)/urdf/scissors_gripper.urdf.xacro"/>
+  <xacro:include filename="$(find ur_robot_driver)/urdf/parallel_gripper.urdf.xacro"/>
   <!-- ros2 control include -->
   <xacro:include filename="$(find ur_robot_driver)/urdf/ur.ros2_control.xacro" />
@@ -101,8 +101,6 @@
   <xacro:arg name="use_mesh" default="true" />
   <xacro:include filename="$(find realsense2_description)/urdf/_d435.urdf.xacro" />
-  <xacro:sensor_d435 parent="tool0" use_nominal_extrinsics="$(arg use_nominal_extrinsics)" add_plug="$(arg add_plug)" use_mesh="$(arg use_mesh)">
-    <!-- TODO: ask vitya for URDF -->
-    <!-- <origin xyz="0.03 0 0.015" rpy="0 -1.57 3.14"/> -->
-    <origin xyz="0.0212132 -0.0212132 0.01" rpy="0 -1.57  2.355"/>
+  <xacro:sensor_d435 parent="gripper_base_link" use_nominal_extrinsics="$(arg use_nominal_extrinsics)" add_plug="$(arg add_plug)" use_mesh="$(arg use_mesh)">
+    <origin xyz="0.0325 -0.0475 0.013" rpy="0 -1.57  1.57"/>
   </xacro:sensor_d435>
 </robot>

Commit message: added pneumatic urdf and behaviour

File: ws/src/Universal_Robots_ROS2_Driver/ur_moveit_config/srdf/ur_macro.srdf.xacro (robot description, xacro)
@@ -14,7 +14,7 @@
       <chain base_link="base_link" tip_link="tool0" />
     </group>
-    <group name="gripper_group">
+    <!-- <group name="gripper_group">
       <joint name="joint_finger_left"/>
-    </group>
+    </group> -->
     <!--GROUP STATES - Purpose - Define a named state for a particular group, in terms of joint values. This is useful to define states like 'folded arms'-->
     <group_state name="home" group="ur_manipulator">

File: ws/src/Universal_Robots_ROS2_Driver/ur_robot_driver/urdf/parallel_gripper.urdf.xacro (robot description, xacro)
@@ -92,5 +92,5 @@
   <joint
     name="joint_finger_right"
-    type="prismatic">
+    type="fixed">
     <origin
       xyz="-0.023845 0 0.0696"
@@ -102,6 +102,6 @@
     <axis
       xyz="1 0 0" />
-    <mimic joint="joint_finger_left" multiplier="1.0"/>
-    <limit lower="0.0" upper="0.023" effort="5.0" velocity="3.0"/>
+    <!-- <mimic joint="joint_finger_left" multiplier="1.0"/> -->
+    <!-- <limit lower="0.0" upper="0.023" effort="5.0" velocity="3.0"/> -->
   </joint>
   <link
@@ -147,5 +147,5 @@
   <joint
     name="joint_finger_left"
-    type="prismatic">
+    type="fixed">
     <origin
       xyz="0.023845 0 0.0696"
@@ -157,5 +157,5 @@
     <axis
       xyz="-1 0 0" />
-    <limit lower="0.0" upper="0.023" effort="5.0" velocity="3.0"/>
+    <!-- <limit lower="0.0" upper="0.023" effort="5.0" velocity="3.0"/> -->
   </joint>
 </robot>

File: ws/src/Universal_Robots_ROS2_Driver/ur_robot_driver/urdf/ur.ros2_control.xacro (robot description, xacro)
@@ -296,8 +296,8 @@
       </gpio>
     </ros2_control>
-    <ros2_control name="ParallelGripperControl" type="system">
+    <!-- <ros2_control name="ParallelGripperControl" type="system">
       <hardware>
         <plugin>feetech_ros2_driver/FeetechHardwareInterface</plugin>
-        <param name="usb_port">/dev/ttyACM1</param>
+        <param name="usb_port">/dev/ttyACM0</param>
       </hardware>
       <joint name="joint_finger_left">
@@ -309,4 +309,17 @@
         <state_interface name="velocity"/>
       </joint>
+    </ros2_control> -->
+    <ros2_control name="SuctionGripperSystem" type="system">
+      <hardware>
+        <plugin>suction_gripper_hardware/SuctionGripperSystem</plugin>
+        <param name="device">/dev/ttyUSB0</param>
+        <param name="baud_rate">115200</param>
+      </hardware>
+      <gpio name="suction_gripper">
+        <command_interface name="state"/>
+        <state_interface name="state">
+          <param name="initial_value">0.0</param>
+        </state_interface>
+      </gpio>
     </ros2_control>
   </xacro:macro>

Commit message: back to parallel gripper || new mid part added

File: ws/src/Universal_Robots_ROS2_Driver/ur_moveit_config/srdf/ur_macro.srdf.xacro (robot description, xacro)
@@ -14,7 +14,7 @@
       <chain base_link="base_link" tip_link="tool0" />
     </group>
-    <!-- <group name="gripper_group">
+    <group name="gripper_group">
       <joint name="joint_finger_left"/>
-    </group> -->
+    </group>
     <!--GROUP STATES - Purpose - Define a named state for a particular group, in terms of joint values. This is useful to define states like 'folded arms'-->
     <group_state name="home" group="ur_manipulator">

File: ws/src/Universal_Robots_ROS2_Driver/ur_robot_driver/urdf/parallel_gripper.urdf.xacro (robot description, xacro)
@@ -92,5 +92,5 @@
   <joint
     name="joint_finger_right"
-    type="fixed">
+    type="prismatic">
     <origin
       xyz="-0.023845 0 0.0696"
@@ -102,6 +102,6 @@
     <axis
       xyz="1 0 0" />
-    <!-- <mimic joint="joint_finger_left" multiplier="1.0"/> -->
-    <!-- <limit lower="0.0" upper="0.023" effort="5.0" velocity="3.0"/> -->
+    <mimic joint="joint_finger_left" multiplier="1.0"/>
+    <limit lower="0.0" upper="0.023" effort="5.0" velocity="3.0"/>
   </joint>
   <link
@@ -147,5 +147,5 @@
   <joint
     name="joint_finger_left"
-    type="fixed">
+    type="prismatic">
     <origin
       xyz="0.023845 0 0.0696"
@@ -157,5 +157,5 @@
     <axis
       xyz="-1 0 0" />
-    <!-- <limit lower="0.0" upper="0.023" effort="5.0" velocity="3.0"/> -->
+    <limit lower="0.0" upper="0.023" effort="5.0" velocity="3.0"/>
   </joint>
 </robot>

File: ws/src/Universal_Robots_ROS2_Driver/ur_robot_driver/urdf/ur.ros2_control.xacro (robot description, xacro)
@@ -296,5 +296,5 @@
       </gpio>
     </ros2_control>
-    <!-- <ros2_control name="ParallelGripperControl" type="system">
+    <ros2_control name="ParallelGripperControl" type="system">
       <hardware>
         <plugin>feetech_ros2_driver/FeetechHardwareInterface</plugin>
@@ -309,6 +309,6 @@
         <state_interface name="velocity"/>
       </joint>
-    </ros2_control> -->
-    <ros2_control name="SuctionGripperSystem" type="system">
+    </ros2_control>
+    <!-- <ros2_control name="SuctionGripperSystem" type="system">
       <hardware>
         <plugin>suction_gripper_hardware/SuctionGripperSystem</plugin>
@@ -322,5 +322,5 @@
         </state_interface>
       </gpio>
-    </ros2_control>
+    </ros2_control> -->
   </xacro:macro>
 </robot>
